File: pcb_v1/pcb_v1.kicad_pcb (KiCad board)
At the start: 2 copper layers, 325.4 x 97.6 mm, 232 parts, among them J1 Conn_01x04, P2 BATT, P3 BATT, SW1 RotaryEncoder, U1 STM32WB55RGVx, U2 SRV05-4, U4 TP4057, U5 XC6206P33

Commit message: New LED Schematic
Parts:
- LED1, LED10, LED11, LED12, LED13, LED14, LED15, LED16, LED17, LED18, LED19, LED2, LED20, LED21, LED22, LED23, LED24, LED25, LED26, LED27, LED28, LED29, LED3, LED30, LED31, LED32, LED33, LED34, LED35, LED36, LED37, LED38, LED39, LED4, LED40, LED41, LED42, LED43, LED44, LED45, LED46, LED47, LED48, LED49, LED5, LED50, LED51, LED52, LED53, LED54, LED55, LED56, LED57, LED58, LED59, LED6, LED60, LED61, LED62, LED63, LED64, LED65, LED66, LED7, LED8, LED9: footprint PCM_marbastlib-mx:LED_MX_6028R -> ScottoKeebs_Components:LED_SK6812MINI
- moved D10 2.26 mm to (103.4, -229.2)
- moved D5 2.21 mm to (8.20, -229.2)
- moved D4 2.21 mm to (-11.0, -229.2)
- moved D7 2.21 mm to (46.2, -229.2)
- moved D1 2.21 mm to (-68.0, -229.4)
- moved D2 2.21 mm to (-49.0, -229.4)
- moved D9 2.20 mm to (84.4, -229.2)
- moved D8 2.05 mm to (65.4, -229.2)
- moved D13 2.01 mm to (160.6, -229.4)
- moved D3 2.01 mm to (-30.0, -229.4)
- moved D6 2.01 mm to (27.2, -229.2)
- moved D11 2.01 mm to (122.4, -229.4)
- moved D12 2.00 mm to (141.6, -229.4)
- moved LED2 0.06 mm to (-57.2, -225.4)
Routing:
- net Row0: track 273.3 -> 228.6 mm
- net Net-(D2-A): track 6.65 -> 12.3 mm
- net Net-(D3-A): track 6.68 -> 11.8 mm
- net Net-(D8-A): track 4.91 -> 9.08 mm
- net Net-(D9-A): track 6.58 -> 8.87 mm
- net Net-(D5-A): track 6.78 -> 8.98 mm
- net Net-(D10-A): track 6.73 -> 8.87 mm
- net Net-(D11-A): track 6.68 -> 8.80 mm
- net Net-(D4-A): track 6.63 -> 8.72 mm
- net Net-(D12-A): track 6.63 -> 8.72 mm
- net Net-(D6-A): track 6.81 -> 8.82 mm
- net Net-(D13-A): track 6.78 -> 8.78 mm
- net Net-(D1-A): track 6.66 -> 8.55 mm
- net Net-(D7-A): track 6.68 -> 8.53 mm

Commit message: Replaced and wired LEDs and Capacitors
Parts:
- added C20: 100nF, Capacitor_SMD:C_0805_2012Metric, B.Cu at (108.8, -225.0)
- added C21: 100nF, Capacitor_SMD:C_0805_2012Metric, B.Cu at (89.8, -225.0)
- added C22: 100nF, Capacitor_SMD:C_0805_2012Metric, B.Cu at (70.8, -225.0)
- added C23: 100nF, Capacitor_SMD:C_0805_2012Metric, B.Cu at (51.8, -225.0)
- added C24: 100nF, Capacitor_SMD:C_0805_2012Metric, B.Cu at (32.6, -225.0)
- added C25: 100nF, Capacitor_SMD:C_0805_2012Metric, B.Cu at (13.6, -225.0)
- added C26: 100nF, Capacitor_SMD:C_0805_2012Metric, B.Cu at (-5.40, -225.0)
- added C27: 100nF, Capacitor_SMD:C_0805_2012Metric, B.Cu at (-24.4, -225.0)
- added C28: 100nF, Capacitor_SMD:C_0805_2012Metric, B.Cu at (-43.4, -225.0)
- added C29: 100nF, Capacitor_SMD:C_0805_2012Metric, B.Cu at (-62.6, -225.1)
- added C30: 100nF, Capacitor_SMD:C_0805_2012Metric, B.Cu at (-81.6, -225.2)
- added C31: 100nF, Capacitor_SMD:C_0805_2012Metric, B.Cu at (61.2, -206.0)
- added C32: 100nF, Capacitor_SMD:C_0805_2012Metric, B.Cu at (42.2, -206.0)
- added C33: 100nF, Capacitor_SMD:C_0805_2012Metric, B.Cu at (23.2, -206.0)
- added C34: 100nF, Capacitor_SMD:C_0805_2012Metric, B.Cu at (4.00, -206.0)
- added C35: 100nF, Capacitor_SMD:C_0805_2012Metric, B.Cu at (-15.0, -206.0)
- added C36: 100nF, Capacitor_SMD:C_0805_2012Metric, B.Cu at (-34.0, -206.0)
- added C37: 100nF, Capacitor_SMD:C_0805_2012Metric, B.Cu at (-53.2, -206.0)
- added C38: 100nF, Capacitor_SMD:C_0805_2012Metric, B.Cu at (-77.0, -206.0)
- added C39: 100nF, Capacitor_SMD:C_0805_2012Metric, B.Cu at (175.6, -225.0)
- added C40: 100nF, Capacitor_SMD:C_0805_2012Metric, B.Cu at (147.0, -225.0)
- added C41: 100nF, Capacitor_SMD:C_0805_2012Metric, B.Cu at (127.8, -225.0)
- added C42: 100nF, Capacitor_SMD:C_0805_2012Metric, B.Cu at (-10.2, -187.0)
- added C43: 100nF, Capacitor_SMD:C_0805_2012Metric, B.Cu at (-29.2, -187.0)
- added C44: 100nF, Capacitor_SMD:C_0805_2012Metric, B.Cu at (-48.2, -187.0)
- added C45: 100nF, Capacitor_SMD:C_0805_2012Metric, B.Cu at (-74.4, -187.0)
- added C46: 100nF, Capacitor_SMD:C_0805_2012Metric, B.Cu at (204.2, -206.0)
- added C47: 100nF, Capacitor_SMD:C_0805_2012Metric, B.Cu at (180.2, -206.0)
- added C48: 100nF, Capacitor_SMD:C_0805_2012Metric, B.Cu at (156.4, -206.2)
- added C49: 100nF, Capacitor_SMD:C_0805_2012Metric, B.Cu at (137.4, -206.0)
- added C50: 100nF, Capacitor_SMD:C_0805_2012Metric, B.Cu at (118.4, -206.2)
- added C51: 100nF, Capacitor_SMD:C_0805_2012Metric, B.Cu at (99.4, -206.0)
- added C52: 100nF, Capacitor_SMD:C_0805_2012Metric, B.Cu at (80.2, -206.0)
- added C53: 100nF, Capacitor_SMD:C_0805_2012Metric, B.Cu at (-69.6, -168.0)
- added C54: 100nF, Capacitor_SMD:C_0805_2012Metric, B.Cu at (204.2, -187.0)
- added C55: 100nF, Capacitor_SMD:C_0805_2012Metric, B.Cu at (173.2, -187.0)
- added C56: 100nF, Capacitor_SMD:C_0805_2012Metric, B.Cu at (142.2, -187.0)
- added C57: 100nF, Capacitor_SMD:C_0805_2012Metric, B.Cu at (123.2, -187.0)
- added C58: 100nF, Capacitor_SMD:C_0805_2012Metric, B.Cu at (104.2, -187.0)
- added C59: 100nF, Capacitor_SMD:C_0805_2012Metric, B.Cu at (85.0, -187.0)
- added C60: 100nF, Capacitor_SMD:C_0805_2012Metric, B.Cu at (66.0, -187.0)
- added C61: 100nF, Capacitor_SMD:C_0805_2012Metric, B.Cu at (47.0, -187.0)
- added C62: 100nF, Capacitor_SMD:C_0805_2012Metric, B.Cu at (28.0, -187.0)
- added C63: 100nF, Capacitor_SMD:C_0805_2012Metric, B.Cu at (8.80, -187.0)
- added C64: 100nF, Capacitor_SMD:C_0805_2012Metric, B.Cu at (158.8, -168.0)
- added C65: 100nF, Capacitor_SMD:C_0805_2012Metric, B.Cu at (132.6, -168.0)
- added C66: 100nF, Capacitor_SMD:C_0805_2012Metric, B.Cu at (113.8, -168.0)
- added C67: 100nF, Capacitor_SMD:C_0805_2012Metric, B.Cu at (94.6, -167.9)
- added C68: 100nF, Capacitor_SMD:C_0805_2012Metric, B.Cu at (75.6, -167.9)
- added C69: 100nF, Capacitor_SMD:C_0805_2012Metric, B.Cu at (56.4, -167.9)
- added C70: 100nF, Capacitor_SMD:C_0805_2012Metric, B.Cu at (37.4, -167.9)
- added C71: 100nF, Capacitor_SMD:C_0805_2012Metric, B.Cu at (18.4, -168.1)
- added C72: 100nF, Capacitor_SMD:C_0805_2012Metric, B.Cu at (-0.60, -167.8)
- added C73: 100nF, Capacitor_SMD:C_0805_2012Metric, B.Cu at (-19.8, -168.0)
- added C74: 100nF, Capacitor_SMD:C_0805_2012Metric, B.Cu at (-38.8, -168.0)
- added C75: 100nF, Capacitor_SMD:C_0805_2012Metric, B.Cu at (204.0, -149.0)
- added C76: 100nF, Capacitor_SMD:C_0805_2012Metric, B.Cu at (185.0, -149.0)
- added C77: 100nF, Capacitor_SMD:C_0805_2012Metric, B.Cu at (166.0, -148.9)
- added C78: 100nF, Capacitor_SMD:C_0805_2012Metric, B.Cu at (135.0, -149.0)
- added C79: 100nF, Capacitor_SMD:C_0805_2012Metric, B.Cu at (111.2, -149.0)
- added C80: 100nF, Capacitor_SMD:C_0805_2012Metric, B.Cu at (39.8, -149.0)
- added C81: 100nF, Capacitor_SMD:C_0805_2012Metric, B.Cu at (-31.6, -149.0)
- added C82: 100nF, Capacitor_SMD:C_0805_2012Metric, B.Cu at (-55.4, -149.0)
- added C83: 100nF, Capacitor_SMD:C_0805_2012Metric, B.Cu at (-79.2, -149.0)
- added C84: 100nF, Capacitor_SMD:C_0805_2012Metric, B.Cu at (204.2, -168.0)
- added C85: 100nF, Capacitor_SMD:C_0805_2012Metric, B.Cu at (185.2, -168.0)
- LED1, LED10, LED11, LED12, LED13, LED14, LED15, LED16, LED17, LED18, LED19, LED2, LED20, LED21, LED22, LED23, LED24, LED25, LED26, LED27, LED28, LED29, LED3, LED30, LED31, LED32, LED33, LED34, LED35, LED36, LED37, LED38, LED39, LED4, LED40, LED41, LED42, LED43, LED44, LED45, LED46, LED47, LED48, LED49, LED5, LED50, LED51, LED52, LED53, LED54, LED55, LED56, LED57, LED58, LED59, LED6, LED60, LED61, LED62, LED63, LED64, LED65, LED66, LED7, LED8, LED9: value MX_LED_6028R -> LED_SK6812MINI
- moved D14 308.6 mm to (188.9, -229.4), turned to 90 degrees
- moved S67 300.5 mm to (152.6, 69.0), turned to 90 degrees
- moved D26 279.7 mm to (150.8, -210.3), turned to 90 degrees
- moved D25 261.8 mm to (131.8, -210.3), turned to 90 degrees
- moved D24 231.2 mm to (112.7, -210.3), turned to 90 degrees
- moved D23 212.7 mm to (93.7, -210.3), turned to 90 degrees
- moved D22 194.3 mm to (74.6, -210.3), turned to 90 degrees
- moved D21 176.0 mm to (55.6, -210.3), turned to 90 degrees
- moved D20 158.1 mm to (36.5, -210.3), turned to 90 degrees
- moved D19 140.5 mm to (17.5, -210.3), turned to 90 degrees
- moved D18 123.5 mm to (-1.59, -210.3), turned to 90 degrees
- moved D17 107.2 mm to (-20.6, -210.3), turned to 90 degrees
- moved D16 92.1 mm to (-39.7, -210.4), turned to 90 degrees
- moved D15 75.5 mm to (-63.5, -210.3), turned to 90 degrees
- moved D61 30.1 mm to (-111.0, -263.5), turned to 90 degrees
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Connections:
- LED1 pad 1: PWRG -> +5V
- LED1 pad 2: PWRR -> Net-(LED1-DOUT)
- LED1 pad 3: PWRB -> GND
- LED1 pad 4: GND -> RGB
- LED10 pad 1: PWRG -> +5V
- LED10 pad 2: PWRR -> Net-(LED10-DOUT)
- LED10 pad 3: PWRB -> GND
- LED10 pad 4: GND -> Net-(LED10-DIN)
- LED11 pad 1: PWRG -> +5V
- LED11 pad 2: PWRR -> Net-(LED11-DOUT)
- LED11 pad 3: PWRB -> GND
- LED11 pad 4: GND -> Net-(LED10-DOUT)
- LED12 pad 1: PWRG -> +5V
- LED12 pad 2: PWRR -> Net-(LED12-DOUT)
- LED12 pad 3: PWRB -> GND
- LED12 pad 4: GND -> Net-(LED11-DOUT)
- LED13 pad 1: PWRG -> +5V
- LED13 pad 2: PWRR -> Net-(LED13-DOUT)
- LED13 pad 3: PWRB -> GND
- LED13 pad 4: GND -> Net-(LED12-DOUT)
- LED14 pad 1: PWRG -> +5V
- LED14 pad 2: PWRR -> Row 1.2
- LED14 pad 3: PWRB -> GND
- LED14 pad 4: GND -> Net-(LED13-DOUT)
- LED15 pad 1: PWRG -> +5V
- LED15 pad 2: PWRR -> Net-(LED15-DOUT)
- LED15 pad 3: PWRB -> GND
- LED15 pad 4: GND -> Row 1.2
- LED16 pad 1: PWRG -> +5V
- LED16 pad 2: PWRR -> Net-(LED16-DOUT)
- LED16 pad 3: PWRB -> GND
- LED16 pad 4: GND -> Net-(LED15-DOUT)
- LED17 pad 1: PWRG -> +5V
- LED17 pad 2: PWRR -> Net-(LED17-DOUT)
- LED17 pad 3: PWRB -> GND
- LED17 pad 4: GND -> Net-(LED16-DOUT)
- LED18 pad 1: PWRG -> +5V
- LED18 pad 2: PWRR -> Net-(LED18-DOUT)
- LED18 pad 3: PWRB -> GND
- LED18 pad 4: GND -> Net-(LED17-DOUT)
- LED19 pad 1: PWRG -> +5V
- LED19 pad 2: PWRR -> Net-(LED19-DOUT)
- LED19 pad 3: PWRB -> GND
- LED19 pad 4: GND -> Net-(LED18-DOUT)
- LED2 pad 1: PWRG -> +5V
- LED2 pad 2: PWRR -> Net-(LED2-DOUT)
- LED2 pad 3: PWRB -> GND
- LED2 pad 4: GND -> Net-(LED1-DOUT)
- LED20 pad 1: PWRG -> +5V
- LED20 pad 2: PWRR -> Net-(LED20-DOUT)
- LED20 pad 3: PWRB -> GND
- LED20 pad 4: GND -> Net-(LED19-DOUT)
- LED21 pad 1: PWRG -> +5V
- LED21 pad 2: PWRR -> Net-(LED21-DOUT)
- LED21 pad 3: PWRB -> GND
- LED21 pad 4: GND -> Net-(LED20-DOUT)
- LED22 pad 1: PWRG -> +5V
- LED22 pad 2: PWRR -> Net-(LED22-DOUT)
- LED22 pad 3: PWRB -> GND
- LED22 pad 4: GND -> Net-(LED21-DOUT)
- LED23 pad 1: PWRG -> +5V
- LED23 pad 2: PWRR -> Net-(LED23-DOUT)
- LED23 pad 3: PWRB -> GND
- LED23 pad 4: GND -> Net-(LED22-DOUT)
- LED24 pad 1: PWRG -> +5V
- LED24 pad 2: PWRR -> Net-(LED24-DOUT)
- LED24 pad 3: PWRB -> GND
- LED24 pad 4: GND -> Net-(LED23-DOUT)
- LED25 pad 1: PWRG -> +5V
- LED25 pad 2: PWRR -> Net-(LED25-DOUT)
- LED25 pad 3: PWRB -> GND
- LED25 pad 4: GND -> Net-(LED24-DOUT)
- LED26 pad 1: PWRG -> +5V
- LED26 pad 2: PWRR -> Net-(LED26-DOUT)
- LED26 pad 3: PWRB -> GND
- LED26 pad 4: GND -> Net-(LED25-DOUT)
- LED27 pad 1: PWRG -> +5V
- LED27 pad 2: PWRR -> Net-(LED27-DOUT)
- LED27 pad 3: PWRB -> GND
- LED27 pad 4: GND -> Net-(LED26-DOUT)
- LED28 pad 1: PWRG -> +5V
- LED28 pad 2: PWRR -> Net-(LED28-DOUT)
- LED28 pad 3: PWRB -> GND
- LED28 pad 4: GND -> Net-(LED27-DOUT)
- LED29 pad 1: PWRG -> +5V
- LED29 pad 2: PWRR -> Row 2.3
- LED29 pad 3: PWRB -> GND
- LED29 pad 4: GND -> Net-(LED28-DOUT)
- LED3 pad 1: PWRG -> +5V
- LED3 pad 2: PWRR -> Net-(LED3-DOUT)
- LED3 pad 3: PWRB -> GND
- LED3 pad 4: GND -> Net-(LED2-DOUT)
- LED30 pad 1: PWRG -> +5V
- LED30 pad 2: PWRR -> Net-(LED30-DOUT)
- LED30 pad 3: PWRB -> GND
- LED30 pad 4: GND -> Row 2.3
- LED31 pad 1: PWRG -> +5V
- LED31 pad 2: PWRR -> Net-(LED31-DOUT)
- LED31 pad 3: PWRB -> GND
- LED31 pad 4: GND -> Net-(LED30-DOUT)
- LED32 pad 1: PWRG -> +5V
- LED32 pad 2: PWRR -> Net-(LED32-DOUT)
- LED32 pad 3: PWRB -> GND
- LED32 pad 4: GND -> Net-(LED31-DOUT)
- LED33 pad 1: PWRG -> +5V
- LED33 pad 2: PWRR -> Net-(LED33-DOUT)
- LED33 pad 3: PWRB -> GND
- LED33 pad 4: GND -> Net-(LED32-DOUT)
- LED34 pad 1: PWRG -> +5V
- LED34 pad 2: PWRR -> Net-(LED34-DOUT)
- LED34 pad 3: PWRB -> GND
- LED34 pad 4: GND -> Net-(LED33-DOUT)
- LED35 pad 1: PWRG -> +5V
- LED35 pad 2: PWRR -> Net-(LED35-DOUT)
- LED35 pad 3: PWRB -> GND
- LED35 pad 4: GND -> Net-(LED34-DOUT)
- LED36 pad 1: PWRG -> +5V
- LED36 pad 2: PWRR -> Net-(LED36-DOUT)
- LED36 pad 3: PWRB -> GND
- LED36 pad 4: GND -> Net-(LED35-DOUT)
- LED37 pad 1: PWRG -> +5V
- LED37 pad 2: PWRR -> Net-(LED37-DOUT)
- LED37 pad 3: PWRB -> GND
- LED37 pad 4: GND -> Net-(LED36-DOUT)
- LED38 pad 1: PWRG -> +5V
- LED38 pad 2: PWRR -> Net-(LED38-DOUT)
- LED38 pad 3: PWRB -> GND
- LED38 pad 4: GND -> Net-(LED37-DOUT)
- LED39 pad 1: PWRG -> +5V
- LED39 pad 2: PWRR -> Net-(LED39-DOUT)
- LED39 pad 3: PWRB -> GND
- LED39 pad 4: GND -> Net-(LED38-DOUT)
- LED4 pad 1: PWRG -> +5V
- LED4 pad 2: PWRR -> Net-(LED4-DOUT)
- LED4 pad 3: PWRB -> GND
- LED4 pad 4: GND -> Net-(LED3-DOUT)
- LED40 pad 1: PWRG -> +5V
- LED40 pad 2: PWRR -> Net-(LED40-DOUT)
- LED40 pad 3: PWRB -> GND
- LED40 pad 4: GND -> Net-(LED39-DOUT)
- LED41 pad 1: PWRG -> +5V
- LED41 pad 2: PWRR -> Net-(LED41-DOUT)
- LED41 pad 3: PWRB -> GND
- LED41 pad 4: GND -> Net-(LED40-DOUT)
- LED42 pad 1: PWRG -> +5V
- LED42 pad 2: PWRR -> Net-(LED42-DOUT)
- LED42 pad 3: PWRB -> GND
- LED42 pad 4: GND -> Net-(LED41-DOUT)
- LED43 pad 1: PWRG -> +5V
- LED43 pad 2: PWRR -> Row 3.4
- LED43 pad 3: PWRB -> GND
- LED43 pad 4: GND -> Net-(LED42-DOUT)
- LED44 pad 1: PWRG -> +5V
- LED44 pad 2: PWRR -> Net-(LED44-DOUT)
- LED44 pad 3: PWRB -> GND
- LED44 pad 4: GND -> Row 3.4
- LED45 pad 1: PWRG -> +5V
- LED45 pad 2: PWRR -> Net-(LED45-DOUT)
- LED45 pad 3: PWRB -> GND
- LED45 pad 4: GND -> Net-(LED44-DOUT)
- LED46 pad 1: PWRG -> +5V
- LED46 pad 2: PWRR -> Net-(LED46-DOUT)
- LED46 pad 3: PWRB -> GND
- LED46 pad 4: GND -> Net-(LED45-DOUT)
- LED47 pad 1: PWRG -> +5V
- LED47 pad 2: PWRR -> Net-(LED47-DOUT)
- LED47 pad 3: PWRB -> GND
- LED47 pad 4: GND -> Net-(LED46-DOUT)
- LED48 pad 1: PWRG -> +5V
- LED48 pad 2: PWRR -> Net-(LED48-DOUT)
- LED48 pad 3: PWRB -> GND
- LED48 pad 4: GND -> Net-(LED47-DOUT)
- LED49 pad 1: PWRG -> +5V
- LED49 pad 2: PWRR -> Net-(LED49-DOUT)
- LED49 pad 3: PWRB -> GND
- LED49 pad 4: GND -> Net-(LED48-DOUT)
- LED5 pad 1: PWRG -> +5V
- LED5 pad 2: PWRR -> Net-(LED5-DOUT)
- LED5 pad 3: PWRB -> GND
- LED5 pad 4: GND -> Net-(LED4-DOUT)
- LED50 pad 1: PWRG -> +5V
- LED50 pad 2: PWRR -> Net-(LED50-DOUT)
- LED50 pad 3: PWRB -> GND
- LED50 pad 4: GND -> Net-(LED49-DOUT)
- LED51 pad 1: PWRG -> +5V
- LED51 pad 2: PWRR -> Net-(LED51-DOUT)
- LED51 pad 3: PWRB -> GND
- LED51 pad 4: GND -> Net-(LED50-DOUT)
- LED52 pad 1: PWRG -> +5V
- LED52 pad 2: PWRR -> Net-(LED52-DOUT)
- LED52 pad 3: PWRB -> GND
- LED52 pad 4: GND -> Net-(LED51-DOUT)
- LED53 pad 1: PWRG -> +5V
- LED53 pad 2: PWRR -> Net-(LED53-DOUT)
- LED53 pad 3: PWRB -> GND
- LED53 pad 4: GND -> Net-(LED52-DOUT)
- LED54 pad 1: PWRG -> +5V
- LED54 pad 2: PWRR -> Net-(LED54-DOUT)
- LED54 pad 3: PWRB -> GND
- LED54 pad 4: GND -> Net-(LED53-DOUT)
- LED55 pad 1: PWRG -> +5V
- LED55 pad 2: PWRR -> Net-(LED55-DOUT)
- LED55 pad 3: PWRB -> GND
- LED55 pad 4: GND -> Net-(LED54-DOUT)
- LED56 pad 1: PWRG -> +5V
- LED56 pad 2: PWRR -> Net-(LED56-DOUT)
- LED56 pad 3: PWRB -> GND
- LED56 pad 4: GND -> Net-(LED55-DOUT)
- LED57 pad 1: PWRG -> +5V
- LED57 pad 2: PWRR -> Row 4.5
- LED57 pad 3: PWRB -> GND
- LED57 pad 4: GND -> Net-(LED56-DOUT)
- LED58 pad 1: PWRG -> +5V
- LED58 pad 2: PWRR -> Net-(LED58-DOUT)
- LED58 pad 3: PWRB -> GND
- LED58 pad 4: GND -> Row 4.5
- LED59 pad 1: PWRG -> +5V
- LED59 pad 2: PWRR -> Net-(LED59-DOUT)
- LED59 pad 3: PWRB -> GND
- LED59 pad 4: GND -> Net-(LED58-DOUT)
- LED6 pad 1: PWRG -> +5V
- LED6 pad 2: PWRR -> Net-(LED6-DOUT)
- LED6 pad 3: PWRB -> GND
- LED6 pad 4: GND -> Net-(LED5-DOUT)
- LED60 pad 1: PWRG -> +5V
- LED60 pad 2: PWRR -> Net-(LED60-DOUT)
- LED60 pad 3: PWRB -> GND
- LED60 pad 4: GND -> Net-(LED59-DOUT)
- LED61 pad 1: PWRG -> +5V
- LED61 pad 2: PWRR -> Net-(LED61-DOUT)
- LED61 pad 3: PWRB -> GND
- LED61 pad 4: GND -> Net-(LED60-DOUT)
- LED62 pad 1: PWRG -> +5V
- LED62 pad 2: PWRR -> Net-(LED62-DOUT)
- LED62 pad 3: PWRB -> GND
- LED62 pad 4: GND -> Net-(LED61-DOUT)
- LED63 pad 1: unconnected-(LED63-GK-Pad1) -> +5V
- LED63 pad 2: unconnected-(LED63-RK-Pad2) -> Net-(LED63-DOUT)
- LED63 pad 3: PWRB -> GND
- LED63 pad 4: GND -> Net-(LED62-DOUT)
- LED64 pad 1: PWRG -> +5V
- LED64 pad 2: PWRR -> Net-(LED64-DOUT)
- LED64 pad 3: PWRB -> GND
- LED64 pad 4: GND -> Net-(LED63-DOUT)
- LED65 pad 1: PWRG -> +5V
- LED65 pad 2: PWRR -> Net-(LED65-DOUT)
- LED65 pad 3: PWRB -> GND
- LED65 pad 4: GND -> Net-(LED64-DOUT)
- LED66 pad 1: PWRG -> +5V
- LED66 pad 2: PWRR -> unconnected-(LED66-DOUT-Pad2)
- LED66 pad 3: PWRB -> GND
- LED66 pad 4: GND -> Net-(LED65-DOUT)
- LED7 pad 1: PWRG -> +5V
- LED7 pad 2: PWRR -> Net-(LED7-DOUT)
- LED7 pad 3: PWRB -> GND
- LED7 pad 4: GND -> Net-(LED6-DOUT)
- LED8 pad 1: PWRG -> +5V
- LED8 pad 2: PWRR -> Net-(LED8-DOUT)
- LED8 pad 3: PWRB -> GND
- LED8 pad 4: GND -> Net-(LED7-DOUT)
- LED9 pad 1: PWRG -> +5V
- LED9 pad 2: PWRR -> Net-(LED10-DIN)
- LED9 pad 3: PWRB -> GND
- LED9 pad 4: GND -> Net-(LED8-DOUT)
Routing:
- net Row1: track 0.00 -> 214.4 mm
- net +5V: track 0.00 -> 180.1 mm
- net Column3: track 327.8 -> 287.4 mm, vias 5 -> 3
- net Column7: track 612.1 -> 572.0 mm, vias 5 -> 3
- net Column5: track 797.7 -> 758.9 mm, vias 7 -> 5
- net Column9: track 469.2 -> 431.7 mm, vias 7 -> 5
- net Row0: track 228.6 -> 256.9 mm
- net Column10: track 395.7 -> 370.9 mm, vias 7 -> 5
- net Column8: track 547.3 -> 535.1 mm, vias 5 -> 3
- net Column6: track 520.8 -> 509.4 mm, vias 5 -> 4
- net Net-(D17-A): track 0.00 -> 8.60 mm
- net Net-(D26-A): track 0.00 -> 8.54 mm
- net Net-(D24-A): track 0.00 -> 8.54 mm
- net Net-(D20-A): track 0.00 -> 8.54 mm
- net Net-(D21-A): track 0.00 -> 8.54 mm
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