File: pcb_v1/pcb_v1.kicad_pcb (KiCad board)
At the start: 2 copper layers, 325.4 x 97.6 mm, 298 parts, among them J1 Conn_01x04, P2 BATT, P3 BATT, SW1 RotaryEncoder, U1 STM32WB55RGVx, U2 SRV05-4, U4 TP4057, U5 XC6206P33

Commit message: Daisy Chained LEDs
Parts:
- moved D57 365.4 mm to (217.4, -172.2)
- moved D66 362.5 mm to (217.6, -153.2)
- moved D43 353.7 mm to (217.4, -191.4)
- moved D29 344.0 mm to (217.8, -211.2)
- moved D56 343.7 mm to (198.4, -172.2)
- moved D65 341.1 mm to (198.4, -153.2)
- moved D42 320.1 mm to (186.6, -191.4)
- moved D64 320.1 mm to (179.4, -153.2)
- moved D28 318.3 mm to (195.8, -215.6)
- moved D55 315.1 mm to (172.2, -172.2)
- moved S67 300.5 mm to (181.0, -230.2), turned to 180 degrees
- moved D27 290.5 mm to (171.2, -215.8)
- moved D63 288.1 mm to (148.4, -153.2)
- moved D54 286.8 mm to (146.0, -172.2)
- moved D41 286.5 mm to (155.6, -191.4)
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Routing:
- net Row 4.5: track 0.00 -> 320.2 mm
- net Row 3.4: track 0.00 -> 320.0 mm
- net Row 2.3: track 0.00 -> 311.6 mm
- net Row4: track 0.00 -> 307.0 mm
- net Row 1.2: track 0.00 -> 285.6 mm
- net Row3: track 0.00 -> 273.8 mm
- net Row2: track 0.00 -> 216.8 mm
- net Net-(LED61-DOUT): track 0.00 -> 80.3 mm
- net Net-(LED60-DOUT): track 0.00 -> 80.2 mm
- net Column9: track 431.7 -> 358.8 mm, vias 5 -> 0
- net Column5: track 758.9 -> 692.3 mm, vias 5 -> 0
- net Column3: track 287.4 -> 235.0 mm, vias 3 -> 0
- net Column7: track 572.0 -> 524.4 mm, vias 3 -> 0
- net Net-(LED42-DOUT): track 0.00 -> 39.8 mm
- net Net-(LED41-DOUT): track 0.00 -> 39.8 mm
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
Commit message: Added 5V connectors to LEDs
Routing:
- net GND: track 0.00 -> 1261.5 mm, vias 0 -> 128
- net +5V: track 180.3 -> 754.1 mm, vias 0 -> 66
- net Column6: track 495.4 -> 139.6 mm
- net Column4: track 268.2 -> 195.7 mm
- net Column8: track 522.2 -> 504.6 mm
- net Column9: track 358.8 -> 357.3 mm
- net Column7: track 524.4 -> 523.1 mm
- net Column10: track 342.4 -> 343.0 mm

Commit message: Drew in Main 5V lines
Routing:
- net +5V: track 754.1 -> 2362.4 mm, vias 66 -> 79
- net Column0: track 0.00 -> 155.9 mm
- net Row 4.5: track 320.2 -> 319.5 mm

Commit message: All 5V LEDs are connected
Parts:
- moved D16 0.16 mm to (-39.7, -210.2)
- moved D15 0.14 mm to (-63.5, -210.2)
Routing:
- net +5V: track 2362.4 -> 2990.0 mm, vias 79 -> 135
- net Column8: track 504.6 -> 495.4 mm, vias 1 -> 0
- net Column4: track 195.7 -> 187.0 mm
- net Column6: track 139.6 -> 135.4 mm, vias 1 -> 0

Commit message: Drew Main Ground Line
Routing:
- net GND: track 1261.5 -> 2808.1 mm, vias 128 -> 135
- net +5V: track 2990.0 -> 2996.9 mm, vias 135 -> 136

Commit message: Fixed Via Sizes
Parts:
- moved J1 56.3 mm to (161.2, -194.1)
- moved D28 5.57 mm to (193.8, -210.4)
- moved D27 5.53 mm to (170.0, -210.4)
- moved D29 0.82 mm to (217.6, -210.4)
Connections:
- C63 pad 2: unconnected-(C63-Pad2) -> GND
- C77 pad 2: unconnected-(C77-Pad2) -> GND
Routing:
- net +5V: track 2996.9 -> 2585.1 mm, vias 136 -> 135
- net Column6: track 135.4 -> 507.0 mm, vias 0 -> 4
- net GND: track 2808.1 -> 2949.9 mm, vias 135 -> 137
- net Column3: track 235.0 -> 121.7 mm
- net Column9: track 357.3 -> 446.6 mm
- net Column7: track 523.1 -> 594.2 mm
- net Row1: track 214.2 -> 281.0 mm
- net Column2: track 0.00 -> 61.9 mm, vias 0 -> 6
- net Column4: track 187.0 -> 149.7 mm, vias 1 -> 0
- net Row2: track 216.8 -> 253.3 mm
- net Column8: track 495.4 -> 523.0 mm, vias 0 -> 4
- net Column5: track 692.3 -> 669.9 mm
- net Net-(D14-A): track 0.00 -> 10.3 mm
- net Net-(D27-A): track 0.00 -> 8.54 mm
- net Net-(D28-A): track 0.00 -> 8.53 mm
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