File: pcb_v1/pcb_v1.kicad_pcb (KiCad board)
At the start: 2 copper layers, 325.4 x 97.6 mm, 298 parts, among them J1 Conn_01x04, P2 BATT, P3 BATT, SW1 RotaryEncoder, U1 STM32WB55RGVx, U2 SRV05-4, U4 TP4057, U5 XC6206P33

Commit message: Clearance fixes
Routing:
- net GND: track 2949.9 -> 2951.5 mm

Commit message: Connected all switches, LEDs to MCU
Parts:
- removed C6, C7, C8: 100nF, Capacitor_SMD:C_0805_2012Metric
- C1, C10, C11, C12, C15, C16, C17, C18, C19, C2, C3, C4, C5, C9, D67, D68, P2, P3, R2, R3, R4, S70, U2, U4, U5: moved to F.Cu
- U1: value STM32WB55RGVx -> STM32WB5MMG; footprint Package_DFN_QFN:QFN-68-1EP_8x8mm_P0.4mm_EP6.4x6.4mm -> PCM_marbastlib-xp-various:STM32WB5MMG
- moved R2 360.1 mm to (64.3, -101.1), turned to 0 degrees
- moved R3 360.1 mm to (64.3, -98.2), turned to 0 degrees
- moved R4 360.1 mm to (64.3, -95.2), turned to 0 degrees
- moved P2 358.0 mm to (68.8, -100.3), turned to 0 degrees
- moved P3 357.8 mm to (56.5, -94.8), turned to 0 degrees
- moved U2 354.2 mm to (64.7, -109.4), turned to 0 degrees
- moved U4 354.2 mm to (64.7, -104.8), turned to 0 degrees
- moved C16 346.0 mm to (59.9, -110.3), turned to 0 degrees
- moved C17 346.0 mm to (59.9, -107.3), turned to 0 degrees
- moved C18 346.0 mm to (59.9, -104.3), turned to 0 degrees
- moved C19 346.0 mm to (59.9, -101.3), turned to 0 degrees
- moved U5 345.9 mm to (68.9, -93.0), turned to 0 degrees
- moved C15 344.7 mm to (55.4, -98.3), turned to 0 degrees
- moved C10 336.7 mm to (55.4, -107.3), turned to 0 degrees
- moved C11 336.7 mm to (55.4, -104.3), turned to 0 degrees
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Connections:
- C12 pad 2: Net-(U1-NRST) -> Net-(U1-PC0)
- C20 pad 1: +5V -> +3.3V
- C21 pad 1: +5V -> +3.3V
- C22 pad 1: +5V -> +3.3V
- C23 pad 1: +5V -> +3.3V
- C24 pad 1: +5V -> +3.3V
- C25 pad 1: +5V -> +3.3V
- C26 pad 1: +5V -> +3.3V
- C27 pad 1: +5V -> +3.3V
- C28 pad 1: +5V -> +3.3V
- C29 pad 1: +5V -> +3.3V
- C30 pad 1: +5V -> +3.3V
- C31 pad 1: +5V -> +3.3V
- C32 pad 1: +5V -> +3.3V
- C33 pad 1: +5V -> +3.3V
- C34 pad 1: +5V -> +3.3V
- C35 pad 1: +5V -> +3.3V
- C36 pad 1: +5V -> +3.3V
- C37 pad 1: +5V -> +3.3V
- C38 pad 1: +5V -> +3.3V
- C39 pad 1: +5V -> +3.3V
- C40 pad 1: +5V -> +3.3V
- C41 pad 1: +5V -> +3.3V
- C42 pad 1: +5V -> +3.3V
- C43 pad 1: +5V -> +3.3V
- C44 pad 1: +5V -> +3.3V
- C45 pad 1: +5V -> +3.3V
- C46 pad 1: +5V -> +3.3V
- C47 pad 1: +5V -> +3.3V
- C48 pad 1: +5V -> +3.3V
- C49 pad 1: +5V -> +3.3V
- C50 pad 1: +5V -> +3.3V
- C51 pad 1: +5V -> +3.3V
- C52 pad 1: +5V -> +3.3V
- C53 pad 1: +5V -> +3.3V
- C54 pad 1: +5V -> +3.3V
- C55 pad 1: +5V -> +3.3V
- C56 pad 1: +5V -> +3.3V
- C57 pad 1: +5V -> +3.3V
- C58 pad 1: +5V -> +3.3V
- C59 pad 1: +5V -> +3.3V
- C60 pad 1: +5V -> +3.3V
- C61 pad 1: +5V -> +3.3V
- C62 pad 1: +5V -> +3.3V
- C63 pad 1: +5V -> +3.3V
- C64 pad 1: +5V -> +3.3V
- C65 pad 1: +5V -> +3.3V
- C66 pad 1: +5V -> +3.3V
- C67 pad 1: +5V -> +3.3V
- C68 pad 1: +5V -> +3.3V
- C69 pad 1: +5V -> +3.3V
- C70 pad 1: +5V -> +3.3V
- C71 pad 1: +5V -> +3.3V
- C72 pad 1: +5V -> +3.3V
- C73 pad 1: +5V -> +3.3V
- C74 pad 1: +5V -> +3.3V
- C75 pad 1: +5V -> +3.3V
- C76 pad 1: +5V -> +3.3V
- C77 pad 1: +5V -> +3.3V
- C78 pad 1: +5V -> +3.3V
- C79 pad 1: +5V -> +3.3V
- C80 pad 1: +5V -> +3.3V
- C81 pad 1: +5V -> +3.3V
- C82 pad 1: +5V -> +3.3V
- C83 pad 1: +5V -> +3.3V
- C84 pad 1: +5V -> +3.3V
- C85 pad 1: +5V -> +3.3V
- LED1 pad 1: +5V -> +3.3V
- LED1 pad 4: RGB -> unconnected-(LED1-DIN-Pad4)
- LED10 pad 1: +5V -> +3.3V
- LED11 pad 1: +5V -> +3.3V
- LED12 pad 1: +5V -> +3.3V
- LED13 pad 1: +5V -> +3.3V
- LED14 pad 1: +5V -> +3.3V
- LED15 pad 1: +5V -> +3.3V
- LED16 pad 1: +5V -> +3.3V
- LED17 pad 1: +5V -> +3.3V
- LED18 pad 1: +5V -> +3.3V
- LED19 pad 1: +5V -> +3.3V
- LED2 pad 1: +5V -> +3.3V
- LED20 pad 1: +5V -> +3.3V
- LED21 pad 1: +5V -> +3.3V
- LED22 pad 1: +5V -> +3.3V
- LED23 pad 1: +5V -> +3.3V
- LED24 pad 1: +5V -> +3.3V
- LED25 pad 1: +5V -> +3.3V
- LED26 pad 1: +5V -> +3.3V
- LED27 pad 1: +5V -> +3.3V
- LED28 pad 1: +5V -> +3.3V
- LED29 pad 1: +5V -> +3.3V
- LED3 pad 1: +5V -> +3.3V
- LED30 pad 1: +5V -> +3.3V
- LED31 pad 1: +5V -> +3.3V
- LED32 pad 1: +5V -> +3.3V
- LED33 pad 1: +5V -> +3.3V
- LED34 pad 1: +5V -> +3.3V
- LED35 pad 1: +5V -> +3.3V
- LED36 pad 1: +5V -> +3.3V
- LED37 pad 1: +5V -> +3.3V
- LED38 pad 1: +5V -> +3.3V
- LED39 pad 1: +5V -> +3.3V
- LED4 pad 1: +5V -> +3.3V
- LED40 pad 1: +5V -> +3.3V
- LED41 pad 1: +5V -> +3.3V
- LED42 pad 1: +5V -> +3.3V
- LED43 pad 1: +5V -> +3.3V
- LED44 pad 1: +5V -> +3.3V
- LED45 pad 1: +5V -> +3.3V
- LED46 pad 1: +5V -> +3.3V
- LED47 pad 1: +5V -> +3.3V
- LED48 pad 1: +5V -> +3.3V
- LED49 pad 1: +5V -> +3.3V
- LED5 pad 1: +5V -> +3.3V
- LED50 pad 1: +5V -> +3.3V
- LED51 pad 1: +5V -> +3.3V
- LED52 pad 1: +5V -> +3.3V
- LED53 pad 1: +5V -> +3.3V
- LED54 pad 1: +5V -> +3.3V
- LED55 pad 1: +5V -> +3.3V
- LED56 pad 1: +5V -> +3.3V
- LED57 pad 1: +5V -> +3.3V
- LED58 pad 1: +5V -> +3.3V
- LED59 pad 1: +5V -> +3.3V
- LED6 pad 1: +5V -> +3.3V
- LED60 pad 1: +5V -> +3.3V
- LED61 pad 1: +5V -> +3.3V
- LED61 pad 2: Net-(LED61-DOUT) -> RGB
- LED62 pad 1: +5V -> +3.3V
- LED62 pad 4: Net-(LED61-DOUT) -> RGB
- LED63 pad 1: +5V -> +3.3V
- LED64 pad 1: +5V -> +3.3V
- LED65 pad 1: +5V -> +3.3V
- LED66 pad 1: +5V -> +3.3V
- LED7 pad 1: +5V -> +3.3V
- LED8 pad 1: +5V -> +3.3V
- LED9 pad 1: +5V -> +3.3V
- U1 pad 1: +3.3V -> unconnected-(U1-PA2-Pad1)
- U1 pad 12: unconnected-(U1-PC3-Pad12) -> Net-(U1-PC0)
- U1 pad 14: +3.3V -> unconnected-(U1-PB8-Pad14)
- U1 pad 15: unconnected-(U1-PA0-Pad15) -> +3.3V
- U1 pad 16: unconnected-(U1-PA1-Pad16) -> GND
- U1 pad 17: unconnected-(U1-PA2-Pad17) -> +3.3V
- U1 pad 18: unconnected-(U1-PA3-Pad18) -> Column7
- U1 pad 19: unconnected-(U1-PA4-Pad19) -> Column8
- U1 pad 20: unconnected-(U1-PA5-Pad20) -> Column9
- U1 pad 21: unconnected-(U1-PA6-Pad21) -> Column10
- U1 pad 22: unconnected-(U1-PA7-Pad22) -> Column11
- U1 pad 23: unconnected-(U1-PA8-Pad23) -> Column12
- U1 pad 24: unconnected-(U1-PA9-Pad24) -> Column13
- U1 pad 25: unconnected-(U1-PC4-Pad25) -> Column14
- U1 pad 30: +3.3V -> unconnected-(U1-PA11/USB-D--Pad30)
- U1 pad 31: unconnected-(U1-RF1-Pad31) -> GND
- U1 pad 32: GND -> unconnected-(U1-VDDUSB-Pad32)
- U1 pad 33: +3.3V -> unconnected-(U1-PD0-Pad33)
- U1 pad 38: unconnected-(U1-PB0-Pad38) -> Row0
- U1 pad 39: unconnected-(U1-PB1-Pad39) -> Row1
- U1 pad 4: unconnected-(U1-PC15-Pad4) -> +3.3V
- U1 pad 40: unconnected-(U1-PE4-Pad40) -> Row2
- U1 pad 42: GND -> unconnected-(U1-PE4-Pad42)
- U1 pad 44: +3.3V -> unconnected-(U1-NC-Pad44)
- U1 pad 45: +3.3V -> Row4
- U1 pad 46: unconnected-(U1-PB12-Pad46) -> Row3
- U1 pad 47: unconnected-(U1-PB13-Pad47) -> Column0
- U1 pad 48: unconnected-(U1-PB14-Pad48) -> Column1
- U1 pad 49: unconnected-(U1-PB15-Pad49) -> Column2
- U1 pad 5: BOOT0 -> GND
- U1 pad 50: unconnected-(U1-PC6-Pad50) -> Column5
- U1 pad 51: unconnected-(U1-PA10-Pad51) -> RGB
- U1 pad 52: D+ -> unconnected-(U1-PA7-Pad52)
- U1 pad 53: D- -> unconnected-(U1-PA6-Pad53)
- U1 pad 54: unconnected-(U1-PA13-Pad54) -> Column3
- U1 pad 55: +3.3V -> Column4
- U1 pad 56: unconnected-(U1-PA14-Pad56) -> Column6
- U1 pad 57: unconnected-(U1-PA15-Pad57) -> GND
- U1 pad 58: unconnected-(U1-PC10-Pad58) -> GND
- U1 pad 59: unconnected-(U1-PC11-Pad59) -> GND
- U1 pad 6: unconnected-(U1-PB8-Pad6) -> +3.3V
- U1 pad 60: unconnected-(U1-PC12-Pad60) -> GND
- U1 pad 67: unconnected-(U1-PB7-Pad67) -> D-
- U1 pad 68: +3.3V -> unconnected-(U1-PD2-Pad68)
- U1 pad 69: GND -> unconnected-(U1-PC9-Pad69)
- U1 pad 8: Net-(U1-NRST) -> unconnected-(U1-PC2-Pad8)
- U1 pad 9: unconnected-(U1-PC0-Pad9) -> BOOT0
Routing:
- net +3.3V: track 0.00 -> 2606.2 mm, vias 0 -> 139
- net +5V: track 2585.1 -> 0.00 mm, vias 135 -> 0
- net Column4: track 150.1 -> 487.0 mm, vias 0 -> 5
- net Column3: track 121.7 -> 405.4 mm, vias 0 -> 5
- net Column11: track 1.82 -> 269.0 mm, vias 0 -> 7
- net Column1: track 0.00 -> 266.5 mm, vias 0 -> 11
- net Column6: track 507.0 -> 747.6 mm, vias 4 -> 7
- net Column2: track 61.9 -> 300.6 mm, vias 6 -> 11
- net Column13: track 0.00 -> 219.1 mm, vias 0 -> 13
- net Column12: track 0.00 -> 214.5 mm, vias 0 -> 3
- net Column14: track 0.00 -> 208.2 mm, vias 0 -> 11
- net Row1: track 281.0 -> 481.3 mm, vias 0 -> 12
- net Row0: track 256.9 -> 449.7 mm, vias 0 -> 10
- net Row2: track 253.3 -> 439.7 mm, vias 0 -> 8
- net Column0: track 156.2 -> 338.6 mm, vias 0 -> 1
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Other:
- board size 325.4 x 97.6 mm -> 325.4 x 98.3 mm

Commit message: Routed trace to rotary encoder
Connections:
- SW1 pad C: Ground -> GND
- U1 pad 52: unconnected-(U1-PA7-Pad52) -> EN1
- U1 pad 53: unconnected-(U1-PA6-Pad53) -> EN2
Routing:
- net EN2: track 0.00 -> 236.4 mm, vias 0 -> 12
- net EN1: track 0.00 -> 233.1 mm, vias 0 -> 12
- net GND: track 3054.7 -> 3076.3 mm
- net Column12: track 214.5 -> 205.4 mm
- net Column0: track 338.6 -> 347.5 mm
- net Row 3.4: track 320.0 -> 314.7 mm
- net Row2: track 439.7 -> 441.9 mm
- net Column13: track 219.1 -> 217.3 mm
- net Row4: track 460.0 -> 461.8 mm
- net Row1: track 481.3 -> 483.0 mm
- net Row 2.3: track 311.6 -> 310.5 mm
- net RGB: track 99.3 -> 100.2 mm
- net Column14: track 208.2 -> 207.5 mm
- net Column11: track 269.0 -> 268.3 mm
- net Row0: track 449.7 -> 449.0 mm
Other:
- board size 325.4 x 98.3 mm -> 353 x 98.7 mm

Commit message: Added Decoupling Capacitors
Parts:
- C1, C10, C11, C12, C15, C16, C17, C18, C19, C2, C3, C4, C5, C9, D67, D68, R2, R3, R4, U2, U4, U5: moved to B.Cu
- moved U5 162.2 mm to (-56.2, -196.1), turned to 90 degrees
- moved C4 66.6 mm to (82.4, -160.0), turned to -90 degrees
- moved C3 60.7 mm to (77.2, -159.0), turned to 180 degrees
- moved C1 60.3 mm to (88.0, -158.0)
- moved C2 60.3 mm to (80.2, -160.0), turned to 90 degrees
- moved C5 57.4 mm to (81.4, -147.0), turned to 180 degrees
- moved C9 52.5 mm to (74.0, -159.4), turned to -90 degrees
- moved C10 51.6 mm to (88.4, -147.0), turned to 180 degrees
- moved C11 47.0 mm to (72.8, -148.0)
- moved P3 43.4 mm to (98.6, -105.4)
- moved P2 35.2 mm to (103.6, -105.7)
- moved U2 13.8 mm to (50.9, -109.4), turned to 180 degrees
- moved U4 13.8 mm to (50.9, -104.8), turned to 180 degrees
- moved R2 13.1 mm to (51.2, -101.1), turned to 180 degrees
- moved R3 13.1 mm to (51.2, -98.2), turned to 180 degrees
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Connections:
- C19 pad 1: 3V3 -> +3.3V
- U1 pad 18: Column7 -> unconnected-(U1-PB7-Pad18)
- U1 pad 19: Column8 -> unconnected-(U1-PB5-Pad19)
- U1 pad 20: Column9 -> unconnected-(U1-PB4-Pad20)
- U1 pad 21: Column10 -> unconnected-(U1-PB3-Pad21)
- U1 pad 22: Column11 -> Column7
- U1 pad 23: Column12 -> Column8
- U1 pad 24: Column13 -> Column9
- U1 pad 25: Column14 -> Column10
- U1 pad 26: unconnected-(U1-PA14/SWCLK-Pad26) -> Column11
- U1 pad 27: unconnected-(U1-PA15-Pad27) -> Column12
- U1 pad 28: unconnected-(U1-PA10-Pad28) -> Column13
- U1 pad 29: unconnected-(U1-PA12/USB-D+-Pad29) -> Column14
- U1 pad 32: unconnected-(U1-VDDUSB-Pad32) -> +3.3V
- U5 pad 2: 3V3 -> +3.3V
Routing:
- net +3.3V: track 2606.2 -> 2666.6 mm, vias 139 -> 144
- net GND: track 3076.3 -> 3082.8 mm, vias 145 -> 146
- net Row2: track 441.9 -> 440.5 mm, vias 8 -> 6
- net EN1: track 233.1 -> 232.1 mm
- net Column8: track 644.5 -> 645.3 mm
- net Column7: track 733.8 -> 734.5 mm
- net Column10: track 402.4 -> 403.1 mm
- net Column12: track 205.4 -> 206.1 mm
- net Column11: track 268.3 -> 268.8 mm
- net Row1: track 483.0 -> 482.6 mm, vias 12 -> 10
- net Row0: vias 10 -> 8
- net RGB: vias 2 -> 4
Other:
- board size 353 x 98.7 mm -> 342.4 x 98.9 mm

Commit message: Added ESP Protection
Parts:
- removed C15: 0.1uF, Capacitor_SMD:C_0805_2012Metric
- removed C16: 10nF, Capacitor_SMD:C_0805_2012Metric
- removed C17, C18, C19: 1uF, Capacitor_SMD:C_0805_2012Metric
- removed D67, D68: B5819W SL, Diode_SMD:D_SOD-123
- removed P2: BATT, Connector_PinHeader_2.54mm:PinHeader_1x02_P2.54mm_Vertical
- removed P3: BATT, Connector_PinSocket_2.00mm:PinSocket_1x02_P2.00mm_Vertical
- removed R2: 4.7K, Resistor_SMD:R_0805_2012Metric
- removed R3: 10M, Resistor_SMD:R_0805_2012Metric
- removed R4: 2.2M, Resistor_SMD:R_0805_2012Metric
- removed U4: TP4057, Package_TO_SOT_SMD:SOT-23-6
- removed U5: XC6206P33, Package_TO_SOT_SMD:SOT-23
- moved S70 163.1 mm to (52.0, 8.98)
- moved U2 67.2 mm to (103.2, -151.6), turned to 0 degrees
- moved C12 56.0 mm to (69.2, -156.6), turned to 0 degrees
- moved C2 22.7 mm to (102.8, -157.6), turned to 180 degrees
- moved C4 0.40 mm to (82.0, -160.0)
Connections:
- U1 pad 21: unconnected-(U1-PB3-Pad21) -> Column7
- U1 pad 22: Column7 -> Column8
- U1 pad 23: Column8 -> Column9
- U1 pad 24: Column9 -> Column10
- U1 pad 25: Column10 -> Column11
- U1 pad 26: Column11 -> Column12
- U1 pad 27: Column12 -> Column13
- U1 pad 28: Column13 -> Column14
- U1 pad 29: Column14 -> VBUS
Routing:
- net VBUS: track 0.00 -> 136.2 mm, vias 0 -> 5
- net GND: track 3082.8 -> 3108.4 mm, vias 146 -> 151
- net Net-(U1-PC0): track 0.00 -> 13.5 mm, vias 0 -> 2
- net D-: track 153.9 -> 163.7 mm, vias 4 -> 5
- net D+: track 162.1 -> 171.7 mm, vias 4 -> 5
- net +3.3V: track 2666.6 -> 2667.3 mm
Other:
- board size 342.4 x 98.9 mm -> 325.4 x 103 mm
