File: esp32_breakout/esp32_breakout_board.kicad_pcb (KiCad board)
At the start: 2 copper layers, 34.7 x 31.8 mm, 12 parts, among them U4 ESP32-S3-MINI-1

Commit message: Updated esp32 breakout board
Parts:
- removed GND2: TestPoint, TestPoint:TestPoint_THTPad_D2.0mm_Drill1.0mm
Routing:
- net GND: track 68.7 -> 60.5 mm
Changed lines of the file:
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@@
-		(embedded_fonts no)
-	)
-	(footprint "TestPoint:TestPoint_THTPad_D2.0mm_Drill1.0mm"
-		(layer "F.Cu")
-		(at 118.8 74)
-		(descr "THT pad as test Point, diameter 2.0mm, hole diameter 1.0mm")
-		(tags "test point THT pad")
-		(property "Reference" "GND2"
-			(at 0 -2.4 0)
-			(layer "F.SilkS")
-			(effects
-				(font
-					(size 1 1)
-					(thickness 0.15)
-				)
-			)
-		)
-		(property "Value" "TestPoint"
-			(at 0 2.05 0)
-			(layer "F.Fab")
-			(hide yes)
-			(effects
-				(font
-					(size 1 1)
-					(thickness 0.15)
-				)
-			)
-		)
-		(property "Datasheet" ""
-			(at 0 0 0)
-			(unlocked yes)
-			(layer "F.Fab")
-			(hide yes)
-			(effects
-				(font
-					(size 1.27 1.27)
-					(thickness 0.15)
-				)
-			)
-		)
-		(property "Description" "test point"
-			(at 0 0 0)
-			(unlocked yes)
-			(layer "F.Fab")
-			(hide yes)
-			(effects
-				(font
-					(size 1.27 1.27)
-					(thickness 0.15)
-				)
-			)
-		)
-		(property ki_fp_filters "Pin* Test*")
-		(sheetname "/")
-		(sheetfile "esp32_breakout_board.kicad_sch")
-		(attr exclude_from_pos_files)
-		(fp_circle
-			(center 0 0)
-			(end 0 1.2)
-			(stroke
-				(width 0.12)
-				(type solid)
-			)
-			(fill no)
-			(layer "F.SilkS")
-		)
-		(fp_circle
-			(center 0 0)
-			(end 1.5 0)
-			(stroke
-				(width 0.05)
-				(type solid)
-			)
-			(fill no)
-			(layer "F.CrtYd")
-		)
-		(pad "1" thru_hole circle
-			(at 0 0)
-			(size 2 2)
-			(drill 1)
-			(layers "*.Cu" "*.Mask")
-			(remove_unused_layers no)
-			(net 1 "GND")
-			(pinfunction "1")
-			(pintype "passive")
-		)
 		(embedded_fonts no)
 	)
@@
 	)
 	(segment
-		(start 122.8 76)
-		(end 126.2 76)
-		(width 0.2)
-		(layer "F.Cu")
-		(net 1)
-	)
-	(segment
 		(start 124.5 77.9)
 		(end 124.4 78)
@@
 	)
 	(segment
-		(start 120.8 74)
-		(end 118.8 74)
-		(width 0.2)
-		(layer "F.Cu")
-		(net 1)
-	)
-	(segment
 		(start 126.2 77.9)
 		(end 124.5 77.9)
@@
 		(layer "F.Cu")
 		(net 1)
-	)
-	(segment
-		(start 120.8 74)
-		(end 122.8 76)
-		(width 0.2)
-		(layer "F.Cu")
-		(net 1)

Commit message: Added silkscreen to boards
Other:
- board text added: "ESP32-S3-Mini-1 UART"
Changed lines of the file:
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@@
 		(layer "Edge.Cuts")
+	)
+	(gr_text "ESP32-S3-Mini-1 UART"
+		(at 118.4 93.4 0)
+		(layer "F.SilkS")
+		(effects
+			(font
+				(size 1.5 1.5)
+				(thickness 0.3)
+				(bold yes)
+			)
+			(justify left bottom)
+		)
 	)
 	(segment
